File: pcb/wordclock2.sch (KiCad schematic (older format))
At the start: 48 parts, among them J1 Jack-DC, J2 CONN_02X05, J3 Micro_SD_Card_Det, J4 USB_OTG, J5 CONN_01X03, J6 CONN_01X03, Q1 FDS6890A, SW1 SW_Push, SW2 SW_Push, SW3 SW_Push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

Commit message: progress
Parts:
- J3: footprint (none) -> wordclockFB:DM3D-SF
- JP1: footprint (none) -> wordclockFB:SOLDER-JUMPER_1-WAY

Commit message: progress
Parts:
- J2: footprint (none) -> wordclockFB:SHF-105-01-L-D-RA
Changed lines of the file:
@@
 F 0 "J2" H 4900 1200 50  0000 C CNN
 F 1 "CONN_02X05" H 4900 600 50  0000 C CNN
-F 2 "" H 4900 -300 50  0001 C CNN
+F 2 "wordclockFB:SHF-105-01-L-D-RA" H 4900 -300 50  0001 C CNN
 F 3 "" H 4900 -300 50  0001 C CNN
 	1    4900 900

Commit message: progress
Parts:
- SW1, SW4: footprint (none) -> Buttons_Switches_SMD:SW_SPST_KMR2
- SW2, SW3: footprint (none) -> Buttons_Switches_ThroughHole:SW_Tactile_SPST_Angled_PTS645Vx39-2LFS
- Y1: footprint (none) -> Crystals:Crystal_SMD_HC49-SD_HandSoldering
- Y2: footprint (none) -> Crystals:Crystal_SMD_SeikoEpson_MC306-4pin_8.0x3.2mm_HandSoldering
Changed lines of the file:
@@
 F 0 "Y2" H 4300 2300 50  0000 C CNN
 F 1 "32.768kHz" H 4300 2000 50  0000 C CNN
-F 2 "" H 4300 2150 50  0001 C CNN
+F 2 "Crystals:Crystal_SMD_SeikoEpson_MC306-4pin_8.0x3.2mm_HandSoldering" H 4300 2150 50  0001 C CNN
 F 3 "" H 4300 2150 50  0001 C CNN
 	1    4300 2150
@@
 F 0 "Y1" H 3550 2750 50  0000 C CNN
 F 1 "8MHz" H 3550 2450 50  0000 C CNN
-F 2 "" H 3550 2600 50  0001 C CNN
+F 2 "Crystals:Crystal_SMD_HC49-SD_HandSoldering" H 3550 2600 50  0001 C CNN
 F 3 "" H 3550 2600 50  0001 C CNN
 	1    3550 2600
@@
 F 0 "SW1" H 1350 3200 50  0000 L CNN
 F 1 "SW_Push" H 1300 3040 50  0000 C CNN
-F 2 "" H 1300 3300 50  0001 C CNN
+F 2 "Buttons_Switches_SMD:SW_SPST_KMR2" H 1300 3300 50  0001 C CNN
 F 3 "" H 1300 3300 50  0001 C CNN
 	1    1300 3100
@@
 F 0 "SW2" H 1350 3450 50  0000 L CNN
 F 1 "SW_Push" H 1300 3290 50  0000 C CNN
-F 2 "" H 1300 3550 50  0001 C CNN
+F 2 "Buttons_Switches_ThroughHole:SW_Tactile_SPST_Angled_PTS645Vx39-2LFS" H 1300 3550 50  0001 C CNN
 F 3 "" H 1300 3550 50  0001 C CNN
 	1    1300 3350
@@
 F 0 "SW3" H 1350 3700 50  0000 L CNN
 F 1 "SW_Push" H 1300 3540 50  0000 C CNN
-F 2 "" H 1300 3800 50  0001 C CNN
+F 2 "Buttons_Switches_ThroughHole:SW_Tactile_SPST_Angled_PTS645Vx39-2LFS" H 1300 3800 50  0001 C CNN
 F 3 "" H 1300 3800 50  0001 C CNN
 	1    1300 3600
@@
 F 0 "SW4" H 11000 6150 50  0000 L CNN
 F 1 "SW_Push" H 10950 5990 50  0000 C CNN
-F 2 "" H 10950 6250 50  0001 C CNN
+F 2 "Buttons_Switches_SMD:SW_SPST_KMR2" H 10950 6250 50  0001 C CNN
 F 3 "" H 10950 6250 50  0001 C CNN
 	1    10950 6050

Commit message: progress
Parts:
- added C14, C15: 100n, Capacitors_SMD:C_0805_HandSoldering, symbol C
- added D3: DIODE, Diodes_SMD:D_PowerDI-123, symbol DIODE
- added R13, R14, R15: 10k, Resistors_SMD:R_0805_HandSoldering, symbol R
- added SW5, SW6: SW_Push, Buttons_Switches_SMD:SW_SPST_KMR2, symbol SW_Push
- C1: footprint (none) -> Capacitors_Tantalum_SMD:CP_Tantalum_Case-D_EIA-7343-31_Hand
- C10, C11, C12, C13, C2, C3, C6, C7, C8, C9: footprint (none) -> Capacitors_SMD:C_0805_HandSoldering
- C4, C5: value 22p -> 33p; footprint (none) -> Capacitors_SMD:C_0805_HandSoldering
- D1, D2: footprint (none) -> LEDs:LED_0805_HandSoldering
- J5, J6: footprint (none) -> wordclockFB:CONN_HEADER_3POS
- R1, R10, R11, R12, R2, R3, R4, R5, R6, R7, R8, R9: footprint (none) -> Resistors_SMD:R_0805_HandSoldering
Connections:
- wire segments 202 -> 216
Other:
- moved on the sheet: C1

Commit message: progress
Parts:
- added C16: 100n, Capacitors_SMD:C_0805_HandSoldering, symbol C
Connections:
- wire segments 216 -> 218

Commit message: battery
Parts:
- BT1: footprint Connect:CR2032H -> wordclockFB:LR44

Commit message: progress, added 32kHz Crystal datasheet
Parts:
- removed Y2: 32.768kHz, Crystals:Crystal_SMD_SeikoEpson_MC306-4pin_8.0x3.2mm_HandSoldering, symbol Crystal
- added Y2: Crystal_GND23, Crystals:Crystal_SMD_SeikoEpson_MC306-4pin_8.0x3.2mm_HandSoldering, symbol Crystal_GND23
- C3: value 1u -> 100n
Connections:
- no-connect marks 19 -> 21
Changed lines of the file:
@@
 	7650 1950 7650 2050
 Connection ~ 7650 2000
-$Comp
-L Crystal Y2
-U 1 1 5983242F
-P 4300 2150
-F 0 "Y2" H 4300 2300 50  0000 C CNN
-F 1 "32.768kHz" H 4300 2000 50  0000 C CNN
-F 2 "Crystals:Crystal_SMD_SeikoEpson_MC306-4pin_8.0x3.2mm_HandSoldering" H 4300 2150 50  0001 C CNN
-F 3 "" H 4300 2150 50  0001 C CNN
-	1    4300 2150
-	0    1    1    0
-$EndComp
 Wire Wire Line
 	5100 2250 4700 2250
@@
 P 2500 7250
 F 0 "C3" H 2525 7350 50  0000 L CNN
-F 1 "1u" H 2525 7150 50  0000 L CNN
+F 1 "100n" H 2525 7150 50  0000 L CNN
 F 2 "Capacitors_SMD:C_0805_HandSoldering" H 2538 7100 50  0001 C CNN
 F 3 "" H 2500 7250 50  0001 C CNN
@@
 	8150 2000 8150 1950
 Connection ~ 7900 2000
+$Comp
+L Crystal_GND23 Y2
+U 1 1 59F49FBD
+P 4300 2150
+F 0 "Y2" H 4425 2350 50  0000 L CNN
+F 1 "Crystal_GND23" H 4425 2275 50  0000 L CNN
+F 2 "Crystals:Crystal_SMD_SeikoEpson_MC306-4pin_8.0x3.2mm_HandSoldering" H 4300 2150 50  0001 C CNN
+F 3 "" H 4300 2150 50  0001 C CNN
+	1    4300 2150
+	0    1    1    0
+$EndComp
+NoConn ~ 4500 2150
+NoConn ~ 4100 2150
 $EndSCHEMATC
