File: pcb/wordclock2.kicad_pcb (KiCad board)
At the start: 2 copper layers, 130 x 30 mm, 57 parts, among them J1 Jack-DC, J2 CONN_02X05, J3 Micro_SD_Card_Det, J4 USB_OTG, J5 CONN_01X03, J6 CONN_01X03, Q1 FDS6890A, SW1 SW_Push, SW2 SW_Push, SW3 SW_Push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

Commit message: first traces
Parts:
- moved R8 14.1 mm to (180.0, 91.6)
- moved BT1 0.25 mm to (150.9, 103.4)
Routing:
- net +5V: track 0.00 -> 149.7 mm, vias 0 -> 2
- net +3V3: track 0.00 -> 107.8 mm, vias 0 -> 4
- net Net-(BZ1-Pad1): track 0.00 -> 34.8 mm
- net /ESP_GPIO0: track 0.00 -> 27.2 mm
- net Net-(C5-Pad2): track 0.00 -> 19.9 mm
- net Net-(R9-Pad2): track 0.00 -> 15.1 mm
- net Net-(R10-Pad2): track 0.00 -> 11.8 mm
- net Net-(C4-Pad2): track 0.00 -> 8.38 mm
- net /UART_OTA_RX: track 0.00 -> 6.74 mm
- net /ST_NRST: track 0.00 -> 3.56 mm
- net /I2C_SCL: track 0.00 -> 3.20 mm
- net /I2C_INT: track 0.00 -> 2.83 mm
- net /I2C_SDA: track 0.00 -> 2.83 mm
Other:
- net class Default: clearance 0.2 -> 0.16; trace_width 0.25 -> 0.16
- net class Power added: clearance 0.16, trace_width 0.16, via_dia 0.6, via_drill 0.4
- rule trace_clearance: 0.2 -> 0.16
- rule trace_min: 0.2 -> 0.16
